Commit message: Removed visual and collison elements for test urdfs

File: test/test_models/meldog_base_link.urdf (robot description, URDF)
Before this commit: robot meldog_core, 18 links, 17 joints
Links:
- link LFF_link: geometry 
- link LFH_link: geometry 
- link LFLL_link: geometry 
- link LFUL_link: geometry 
- link LRF_link: geometry 
- link LRH_link: geometry 
- link LRLL_link: geometry 
- link LRUL_link: geometry 
- link RFF_link: geometry 
- link RFH_link: geometry 
- link RFLL_link: geometry 
- link RFUL_link: geometry 
- link RRF_link: geometry 
- link RRH_link: geometry 
- link RRLL_link: geometry 
- link RRUL_link: geometry 

File: test/test_models/meldog_no_base_link.urdf (robot description, URDF)
Before this commit: robot meldog_core, 17 links, 16 joints
Links:
- link LFF_link: geometry 
- link LFH_link: geometry 
- link LFLL_link: geometry 
- link LFUL_link: geometry 
- link LRF_link: geometry 
- link LRH_link: geometry 
- link LRLL_link: geometry 
- link LRUL_link: geometry 
- link RFF_link: geometry 
- link RFH_link: geometry 
- link RFLL_link: geometry 
- link RFUL_link: geometry 
- link RRF_link: geometry 
- link RRH_link: geometry 
- link RRLL_link: geometry 
- link RRUL_link: geometry 
